Commit message: Added URDF and STL to RVIZ preview
Signed-off-by: Tomer <tomerstein@mail.tau.ac.il>

File: src/arm_description/urdf/Arm_MoveIt_Assembly.SLDASM.urdf (robot description, URDF)
Before this commit: robot Arm_MoveIt_Assembly.SLDASM, 6 links, 5 joints
Links:
- link End_effector: geometry collision mesh filename=package://arm_description/meshes/End_effector.STL; visual mesh filename=package://arm_description/meshes/End_effector.STL
- link base_link: geometry collision mesh filename=package://arm_description/meshes/base_link.STL; visual mesh filename=package://arm_description/meshes/base_link.STL
- link link1: geometry collision mesh filename=package://arm_description/meshes/link1.STL; visual mesh filename=package://arm_description/meshes/link1.STL
- link link2: geometry collision mesh filename=package://arm_description/meshes/link2.STL; visual mesh filename=package://arm_description/meshes/link2.STL
- link link3: geometry collision mesh filename=package://arm_description/meshes/link3.STL; visual mesh filename=package://arm_description/meshes/link3.STL
- link link4: geometry collision mesh filename=package://arm_description/meshes/link4.STL; visual mesh filename=package://arm_description/meshes/link4.STL

Commit message: Added limits to joints
Signed-off-by: Tomer <tomerstein@mail.tau.ac.il>

File: src/arm_description/urdf/Arm_MoveIt_Assembly.SLDASM.urdf (robot description, URDF)
Before this commit: robot Arm_MoveIt_Assembly.SLDASM, 6 links, 5 joints
Joints:
- joint Joint1: limit lower=0 upper=0 effort=0 velocity=0 -> lower=-1 upper=1 effort=0 velocity=0
- joint Joint2: limit lower=0 upper=0 effort=0 velocity=0 -> lower=-1 upper=1 effort=0 velocity=0
- joint Joint3: limit lower=0 upper=0 effort=0 velocity=0 -> lower=-1 upper=1 effort=0 velocity=0
- joint Joint4: limit lower=0 upper=0 effort=0 velocity=0 -> lower=-1 upper=1 effort=0 velocity=0

Commit message: latest srdf / urdf

File: src/arm_description/urdf/Arm_MoveIt_Assembly.SLDASM.urdf (robot description, URDF)
Before this commit: robot Arm_MoveIt_Assembly.SLDASM, 6 links, 5 joints
Joints:
- joint Joint1: limit lower=-1 upper=1 effort=0 velocity=0 -> lower=-3 upper=3 effort=0 velocity=0
- joint Joint2: limit lower=-1 upper=1 effort=0 velocity=0 -> lower=-3 upper=3 effort=0 velocity=0
- joint Joint3: limit lower=-1 upper=1 effort=0 velocity=0 -> lower=-3 upper=3 effort=0 velocity=0
- joint Joint4: limit lower=-1 upper=1 effort=0 velocity=0 -> lower=-3 upper=3 effort=0 velocity=0

File: src/arm_description/urdf/arm.urdf.xacro (robot description, xacro)
@@ -76,5 +76,5 @@
     <origin xyz="0 0 0.2" rpy="0 0 0"/>
     <axis xyz="0 1 0"/>
-    <limit lower="-1.57" upper="1.57" effort="15.0" velocity="12.0"/>
+    <limit lower="-3.14" upper="3.14" effort="15.0" velocity="12.0"/>
   </joint>
   <link name="link3">
@@ -98,5 +98,5 @@
     <origin xyz="0 0 0.2" rpy="0 0 0"/>
     <axis xyz="0 1 0"/>
-    <limit lower="-1.57" upper="1.57" effort="15.0" velocity="12.0"/>
+    <limit lower="-3.14" upper="3.14" effort="15.0" velocity="12.0"/>
   </joint>
   <link name="link4">
@@ -146,5 +146,5 @@
     <origin xyz="0 0 0.1" rpy="0 0 0"/>
     <axis xyz="0 1 0"/>
-    <limit lower="-1.57" upper="1.57" effort="5.0" velocity="17.5"/>
+    <limit lower="-3.14" upper="3.14" effort="5.0" velocity="17.5"/>
   </joint>
   <!-- End effector link -->

Commit message: change the end- effector in the URDF Signed-off-by: Omri Talmon <omritalmon@mail.tau.ac.il>

File: src/arm_description/urdf/Arm_MoveIt_Assembly.SLDASM.urdf (robot description, URDF)
Before this commit: robot Arm_MoveIt_Assembly.SLDASM, 6 links, 5 joints
Joints:
- joint end_effector: axis 0 0 0 -> 0 0 -1; limit (none) -> lower=0 upper=0 effort=0 velocity=0; type fixed -> revolute

Commit message: UPDATED CODE
Signed-off-by: Yaelc2001 <yaelc2001@gmail.com>

File: src/arm_description/urdf/Arm_MoveIt_Assembly.SLDASM.urdf (robot description, URDF)
Before this commit: robot Arm_MoveIt_Assembly.SLDASM, 6 links, 5 joints
Joints:
- removed joint end_effector
- added joint Joint5: type revolute, parent link4, child End_effector, origin xyz=0 -0.0617 -0.1125 rpy=0 0 0, axis 0 0 -1, limit lower=-3 upper=3 effort=0 velocity=0

Commit message: servo fix
Signed-off-by: Omri Talmon <omritalmon@mail.tau.ac.il>

File: src/arm_description/urdf/Arm_MoveIt_Assembly.SLDASM.urdf (robot description, URDF)
Before this commit: robot Arm_MoveIt_Assembly.SLDASM, 6 links, 5 joints
Joints:
- joint Joint1: limit lower=-2 upper=2 effort=0 velocity=0 -> lower=-10 upper=10 effort=100 velocity=7.5
- joint Joint2: limit lower=-2 upper=2 effort=0 velocity=0 -> lower=-10 upper=10 effort=100 velocity=7.5
- joint Joint3: limit lower=-2 upper=2 effort=0 velocity=0 -> lower=-10 upper=10 effort=100 velocity=7.5
- joint Joint4: limit lower=-2 upper=2 effort=0 velocity=0 -> lower=-10 upper=10 effort=100 velocity=7.5
- joint Joint5: limit lower=-2 upper=2 effort=0 velocity=0 -> lower=-10 upper=10 effort=100 velocity=7.5
