Commit message: working moveit.launch.py

File: src/arm_controller/urdf/cubemars_test.ros2_control.urdf.xacro (robot description, xacro)
@@ -9,5 +9,5 @@
     </hardware>
     <!-- Five actuator joints with CAN IDs 30-34 -->
-    <joint name="joint1">
+    <joint name="Joint1">
       <param name="can_id">30</param>      <!-- CAN ID 30 (0x1E) -->
       <param name="pole_pairs">21</param>
@@ -23,5 +23,5 @@
       <state_interface name="effort"/>
     </joint>
-    <joint name="joint2">
+    <joint name="Joint2">
       <param name="can_id">31</param>      <!-- CAN ID 31 (0x1F) -->
       <param name="pole_pairs">21</param>
@@ -37,5 +37,5 @@
       <state_interface name="effort"/>
     </joint>
-    <joint name="joint3">
+    <joint name="Joint3">
       <param name="can_id">32</param>      <!-- CAN ID 32 (0x20) -->
       <param name="pole_pairs">21</param>
@@ -51,5 +51,5 @@
       <state_interface name="effort"/>
     </joint>
-    <joint name="joint4">
+    <joint name="Joint4">
       <param name="can_id">33</param>      <!-- CAN ID 33 (0x21) -->
       <param name="pole_pairs">21</param>
@@ -65,5 +65,5 @@
       <state_interface name="effort"/>
     </joint>
-    <joint name="joint5">
+    <joint name="Joint5">
       <param name="can_id">34</param>      <!-- CAN ID 34 (0x22) -->
       <param name="pole_pairs">21</param>

File: src/arm_description/urdf/arm.ros2_control.xacro (robot description, xacro)
@@ -15,5 +15,5 @@
       </hardware>
       <!-- Joint 1 -->
-      <joint name="joint1">
+      <joint name="Joint1">
         <param name="can_id">30</param>
         <param name="pole_pairs">21</param>
@@ -30,5 +30,5 @@
       </joint>
       <!-- Joint 2 -->
-      <joint name="joint2">
+      <joint name="Joint2">
         <param name="can_id">31</param>
         <param name="pole_pairs">21</param>
@@ -45,5 +45,5 @@
       </joint>
       <!-- Joint 3 -->
-      <joint name="joint3">
+      <joint name="Joint3">
         <param name="can_id">32</param>
         <param name="pole_pairs">21</param>
@@ -60,5 +60,5 @@
       </joint>
       <!-- Joint 4 -->
-      <joint name="joint4">
+      <joint name="Joint4">
         <param name="can_id">33</param>
         <param name="pole_pairs">21</param>
@@ -75,5 +75,5 @@
       </joint>
       <!-- Joint 5 -->
-      <joint name="joint5">
+      <joint name="Joint5">
         <param name="can_id">34</param>
         <param name="pole_pairs">21</param>

File: src/arm_description/urdf/arm.urdf.xacro (robot description, xacro)
@@ -1,3 +1,3 @@
-<!-- <?xml version="1.0"?>
+<?xml version="1.0"?>
 <robot name="exodus_arm" xmlns:xacro="http://www.ros.org/wiki/xacro">
   <!-- TODO: Add actual URDF description here omri and tomer this is a structure example -->
@@ -156,3 +156,2 @@
   </joint>
 </robot>
- -->

Commit message: Changed motors limits for Moveit2 Also changed gear ratio to motors ID 31, 32
Signed-off-by: Omri Talmon <omritalmon@mail.tau.ac.il>

File: src/arm_controller/urdf/cubemars_test.ros2_control.urdf.xacro (robot description, xacro)
@@ -26,5 +26,5 @@
       <param name="can_id">31</param>      <!-- CAN ID 31 (0x1F) -->
       <param name="pole_pairs">21</param>
-      <param name="gear_ratio">64</param>
+      <param name="gear_ratio">1</param>
       <param name="kt">0.105</param>
       <param name="vel_limit">12.0</param>

File: src/arm_description/urdf/Arm_MoveIt_Assembly.SLDASM.urdf (robot description, URDF)
Before this commit: robot Arm_MoveIt_Assembly.SLDASM, 6 links, 5 joints
Joints:
- joint Joint1: limit lower=-3 upper=3 effort=0 velocity=0 -> lower=-2 upper=2 effort=0 velocity=0
- joint Joint2: limit lower=-3 upper=3 effort=0 velocity=0 -> lower=-2 upper=2 effort=0 velocity=0
- joint Joint3: limit lower=-3 upper=3 effort=0 velocity=0 -> lower=-2 upper=2 effort=0 velocity=0
- joint Joint4: limit lower=-3 upper=3 effort=0 velocity=0 -> lower=-2 upper=2 effort=0 velocity=0
- joint Joint5: limit lower=-3 upper=3 effort=0 velocity=0 -> lower=-2 upper=2 effort=0 velocity=0

File: src/arm_description/urdf/arm.ros2_control.xacro (robot description, xacro)
@@ -33,5 +33,5 @@
         <param name="can_id">31</param>
         <param name="pole_pairs">21</param>
-        <param name="gear_ratio">64</param>
+        <param name="gear_ratio">1</param>
         <param name="kt">0.105</param>
         <param name="vel_limit">12.0</param>

File: src/arm_description/urdf/arm.urdf.xacro (robot description, xacro)
@@ -53,5 +53,5 @@
     <child link="link1" />
     <axis xyz="0 0 1" />
-    <limit lower="-3" upper="3" effort="0" velocity="0" />
+    <limit lower="-10" upper="10" effort="0" velocity="0" />
   </joint>
   <link name="link2">
@@ -82,5 +82,5 @@
     <child link="link2" />
     <axis xyz="0 -1 0" />
-    <limit lower="-3" upper="3" effort="0" velocity="0" />
+    <limit lower="-10" upper="10" effort="0" velocity="0" />
   </joint>
   <link name="link3">
@@ -111,5 +111,5 @@
     <child link="link3" />
     <axis xyz="0 1 0" />
-    <limit lower="-3" upper="3" effort="0" velocity="0" />
+    <limit lower="-10" upper="10" effort="0" velocity="0" />
   </joint>
   <link name="link4">
@@ -140,5 +140,5 @@
     <child link="link4" />
     <axis xyz="0 -1 0" />
-    <limit lower="-3" upper="3" effort="0" velocity="0" />
+    <limit lower="-10" upper="10" effort="0" velocity="0" />
   </joint>
   <link name="End_effector">
@@ -169,5 +169,5 @@
     <child link="End_effector" />
     <axis xyz="0 0 -1" />
-    <limit lower="-3" upper="3" effort="0" velocity="0" />
+    <limit lower="-10" upper="10" effort="0" velocity="0" />
   </joint>
   <xacro:arm_ros2_control

Commit message: moving arm + gripper patch final working stable model
Signed-off-by: TAUverIL <TAUverIL@gmail.com>

File: src/arm_controller/urdf/cubemars_test.ros2_control.urdf.xacro (robot description, xacro)
@@ -26,7 +26,8 @@
       <param name="can_id">31</param>      <!-- CAN ID 31 (0x1F) -->
       <param name="pole_pairs">21</param>
-      <param name="gear_ratio">1</param>
+      <param name="gear_ratio">64</param>
       <param name="kt">0.105</param>
-      <param name="vel_limit">12.0</param>
+      <param name="vel_limit">5.03</param>
+      <param name="trq_limit">120</param>
       <param name="acc_limit">3.0</param>
       <param name="enc_off">0.0</param>

File: src/arm_controller/urdf/dynamixel_test.ros2_control.urdf.xacro (robot description, xacro)
@@ -2,5 +2,5 @@
 <robot xmlns:xacro="http://www.ros.org/wiki/xacro" name="dynamixel_test_robot">
   <link name="world"/>
-  <link name="link1">
+  <link name="Link_5">
     <inertial>
       <mass value="0.1"/>
@@ -9,9 +9,35 @@
     </inertial>
   </link>
-  <joint name="joint1" type="revolute">
+  <link name="Finger_Left">
+    <inertial>
+      <mass value="0.05"/>
+      <origin xyz="0 0 0"/>
+      <inertia ixx="0.001" ixy="0" ixz="0" iyy="0.001" iyz="0" izz="0.001"/>
+    </inertial>
+  </link>
+  <link name="Finger_Right">
+    <inertial>
+      <mass value="0.05"/>
+      <origin xyz="0 0 0"/>
+      <inertia ixx="0.001" ixy="0" ixz="0" iyy="0.001" iyz="0" izz="0.001"/>
+    </inertial>
+  </link>
+  <joint name="world_to_link5" type="fixed">
     <parent link="world"/>
-    <child link="link1"/>
-    <axis xyz="0 0 1"/>
-    <limit lower="-3.14" upper="3.14" effort="10.0" velocity="5.0"/>
+    <child link="Link_5"/>
+    <origin xyz="0 0 0" rpy="0 0 0"/>
+  </joint>
+  <joint name="Finger_Left_Joint" type="prismatic">
+    <parent link="Link_5"/>
+    <child link="Finger_Left"/>
+    <axis xyz="-1 0 0"/>
+    <limit lower="0.0" upper="0.04" effort="7.3" velocity="5.55"/>
+  </joint>
+  <joint name="Finger_Right_Joint" type="prismatic">
+    <parent link="Link_5"/>
+    <child link="Finger_Right"/>
+    <axis xyz="1 0 0"/>
+    <limit lower="0.0" upper="0.04" effort="7.3" velocity="5.55"/>
+    <mimic joint="Finger_Left_Joint"/>
   </joint>
   <ros2_control name="DynamixelSystem" type="system">
@@ -21,5 +47,5 @@
       <param name="baud_rate">57600</param>
     </hardware>
-    <joint name="joint1">
+    <joint name="Finger_Left_Joint">
       <param name="id">1</param>
       <command_interface name="position"/>

File: src/arm_description/urdf/arm.ros2_control.xacro (robot description, xacro)
@@ -1,5 +1,5 @@
 <?xml version="1.0"?>
 <robot xmlns:xacro="http://www.ros.org/wiki/xacro">
-  <xacro:macro name="arm_ros2_control" params="name use_fake_hardware:=false can_interface:=slcan0">
+  <xacro:macro name="arm_ros2_control" params="name use_fake_hardware:=false can_interface:=slcan0 use_gripper:=false">
     <ros2_control name="${name}" type="system">
       <hardware>
@@ -15,5 +15,5 @@
       </hardware>
       <!-- Joint 1 -->
-      <joint name="Joint1">
+      <joint name="Joint_1">
         <param name="can_id">30</param>
         <param name="pole_pairs">21</param>
@@ -30,5 +30,5 @@
       </joint>
       <!-- Joint 2 -->
-      <joint name="Joint2">
+      <joint name="Joint_2">
         <param name="can_id">31</param>
         <param name="pole_pairs">21</param>
@@ -38,4 +38,5 @@
         <param name="acc_limit">3.0</param>
         <param name="enc_off">0.0</param>
+        <param name="direction">-1</param>
         <param name="read_only">0</param>
         <command_interface name="position"/>
@@ -45,10 +46,10 @@
       </joint>
       <!-- Joint 3 -->
-      <joint name="Joint3">
+      <joint name="Joint_3">
         <param name="can_id">32</param>
         <param name="pole_pairs">21</param>
         <param name="gear_ratio">64</param>
         <param name="kt">0.105</param>
-        <param name="vel_limit">12.0</param>
+        <param name="vel_limit">5.03</param>
         <param name="acc_limit">3.0</param>
         <param name="enc_off">0.0</param>
@@ -60,5 +61,5 @@
       </joint>
       <!-- Joint 4 -->
-      <joint name="Joint4">
+      <joint name="Joint_4">
         <param name="can_id">33</param>
         <param name="pole_pairs">21</param>
@@ -66,5 +67,5 @@
         <param name="kt">0.1</param>
         <param name="vel_limit">2.5</param>
-        <param name="acc_limit">10.0</param>
+        <param name="acc_limit">5.0</param>
         <param name="enc_off">0.0</param>
         <param name="read_only">0</param>
@@ -75,5 +76,5 @@
       </joint>
       <!-- Joint 5 -->
-      <joint name="Joint5">
+      <joint name="Joint_5">
         <param name="can_id">34</param>
         <param name="pole_pairs">21</param>
@@ -90,4 +91,30 @@
       </joint>
     </ros2_control>
+    <xacro:if value="${use_gripper}">
+      <ros2_control name="DynamixelSystem" type="system">
+        <hardware>
+          <xacro:if value="${use_fake_hardware}">
+            <plugin>mock_components/GenericSystem</plugin>
+          </xacro:if>
+          <xacro:unless value="${use_fake_hardware}">
+            <plugin>dynamixel_interface/DynamixelSystem</plugin>
+            <param name="device_name">/dev/ttyUSB0</param>
+            <param name="baud_rate">57600</param>
+          </xacro:unless>
+        </hardware>
+        <!-- Gripper Left Finger -->
+        <joint name="Finger_Left_Joint">
+          <param name="id">1</param>
+          <!-- Map MoveIt/URDF gripper travel to calibrated Dynamixel motor radians.
+               URDF: 0.0 = closed, 0.04 = open. Dynamixel: 0.5 = closed, -1.9 = open. -->
+          <param name="position_to_motor_scale">-60.0</param>
+          <param name="position_to_motor_offset">0.5</param>
+          <command_interface name="position"/>
+          <state_interface name="position"/>
+          <state_interface name="velocity"/>
+          <state_interface name="effort"/>
+        </joint>
+      </ros2_control>
+    </xacro:if>
   </xacro:macro>
 </robot>

File: src/arm_description/urdf/arm.urdf.xacro (robot description, xacro)
@@ -3,175 +3,38 @@
   <xacro:arg name="use_fake_hardware" default="false"/>
   <xacro:arg name="can_interface" default="slcan0"/>
+  <xacro:arg name="use_gripper" default="false"/>
+  <xacro:include filename="$(find arm_description)/urdf/AssemblyURDF_27.04.26.urdf"/>
   <xacro:include filename="$(find arm_description)/urdf/arm.ros2_control.xacro"/>
-  <link name="base_link">
-    <inertial>
-      <origin xyz="-1.60427944681102E-05 3.87300953518382E-05 0.0414251446336533" rpy="0 0 0" />
-      <mass value="0.655014596547137" />
-      <inertia ixx="0.00101073031912522" ixy="-1.90767935198547E-07" ixz="-1.70165593174546E-07" iyy="0.00095401536565403" iyz="4.10819611617684E-07" izz="0.00188699356120778" />
-    </inertial>
+  <xacro:arm_ros2_control
+    name="ExodusArmSystem"
+    use_fake_hardware="$(arg use_fake_hardware)"
+    can_interface="$(arg can_interface)"
+    use_gripper="$(arg use_gripper)"/>
+  <!-- Camera Attached to Link_3 -->
+  <link name="camera_link">
     <visual>
-      <origin xyz="0 0 0" rpy="0 0 0" />
       <geometry>
-        <mesh filename="package://arm_description/meshes/base_link.STL" />
+        <box size="0.04 0.1 0.04"/>
       </geometry>
-      <material name="">
-        <color rgba="0.792156862745098 0.819607843137255 0.933333333333333 1" />
+      <material name="camera_material">
+        <color rgba="0.2 0.2 0.2 1.0"/>
       </material>
     </visual>
     <collision>
-      <origin xyz="0 0 0" rpy="0 0 0" />
       <geometry>
-        <mesh filename="package://arm_description/meshes/base_link.STL" />
+        <box size="0.04 0.1 0.04"/>
       </geometry>
     </collision>
+    <inertial>
+      <mass value="0.1"/>
+      <origin xyz="0 0 0"/>
+      <inertia ixx="0.0001" ixy="0" ixz="0" iyy="0.0001" iyz="0" izz="0.0001"/>
+    </inertial>
   </link>
-  <link name="link1">
-    <inertial>
-      <origin xyz="-2.98433441166951E-05 -0.0483515314635655 0.054713057999731" rpy="0 0 0" />
-      <mass value="0.455125224183725" />
-      <inertia ixx="0.000394829058309459" ixy="-3.74478064371689E-07" ixz="-3.68999770581118E-07" iyy="0.000530839403055201" iyz="2.00439805340242E-05" izz="0.000397964515551658" />
-    </inertial>
-    <visual>
-      <origin xyz="0 0 0" rpy="0 0 0" />
-      <geometry>
-        <mesh filename="package://arm_description/meshes/link1.STL" />
-      </geometry>
-      <material name="">
-        <color rgba="0.792156862745098 0.819607843137255 0.933333333333333 1" />
-      </material>
-    </visual>
-    <collision>
-      <origin xyz="0 0 0" rpy="0 0 0" />
-      <geometry>
-        <mesh filename="package://arm_description/meshes/link1.STL" />
-      </geometry>
-    </collision>
-  </link>
-  <joint name="Joint1" type="revolute">
-    <origin xyz="0 0 0.0775" rpy="0 0 0" />
-    <parent link="base_link" />
-    <child link="link1" />
-    <axis xyz="0 0 1" />
-    <limit lower="-10" upper="10" effort="0" velocity="0" />
+  <joint name="camera_joint" type="fixed">
+    <parent link="Link_3"/>
+    <child link="camera_link"/>
+    <!-- Position the camera in the middle of Link_3 (which is ~0.45m long along -X) and slightly above it -->
+    <origin xyz="-0.226 0.0 0.08" rpy="0 0 0"/>
   </joint>
-  <link name="link2">
-    <inertial>
-      <origin xyz="9.27579481573709E-05 0.0175182399290933 0.275472999386939" rpy="0 0 0" />
-      <mass value="0.891856461721987" />
-      <inertia ixx="0.00435475407288075" ixy="-1.03883193767188E-07" ixz="-2.20593156848708E-07" iyy="0.0045575625095459" iyz="-2.0247268665606E-06" izz="0.000474727840907135" />
-    </inertial>
-    <visual>
-      <origin xyz="0 0 0" rpy="0 0 0" />
-      <geometry>
-        <mesh filename="package://arm_description/meshes/link2.STL" />
-      </geometry>
-      <material name="">
-        <color rgba="0.792156862745098 0.819607843137255 0.933333333333333 1" />
-      </material>
-    </visual>
-    <collision>
-      <origin xyz="0 0 0" rpy="0 0 0" />
-      <geometry>
-        <mesh filename="package://arm_description/meshes/link2.STL" />
-      </geometry>
-    </collision>
-  </link>
-  <joint name="Joint2" type="revolute">
-    <origin xyz="0 -0.024 0.06" rpy="0 0 0" />
-    <parent link="link1" />
-    <child link="link2" />
-    <axis xyz="0 -1 0" />
-    <limit lower="-10" upper="10" effort="0" velocity="0" />
-  </joint>
-  <link name="link3">
-    <inertial>
-      <origin xyz="-0.279853886139342 0.0148848609580054 -8.90398865749376E-14" rpy="0 0 0" />
-      <mass value="0.820660258517619" />
-      <inertia ixx="0.000344535085998629" ixy="-4.48152667831305E-07" ixz="-2.93896707624529E-09" iyy="0.00648723879471234" iyz="-1.18705365636058E-19" izz="0.00626772615915786" />
-    </inertial>
-    <visual>
-      <origin xyz="0 0 0" rpy="0 0 0" />
-      <geometry>
-        <mesh filename="package://arm_description/meshes/link3.STL" />
-      </geometry>
-      <material name="">
-        <color rgba="0.792156862745098 0.819607843137255 0.933333333333333 1" />
-      </material>
-    </visual>
-    <collision>
-      <origin xyz="0 0 0" rpy="0 0 0" />
-      <geometry>
-        <mesh filename="package://arm_description/meshes/link3.STL" />
-      </geometry>
-    </collision>
-  </link>
-  <joint name="Joint3" type="revolute">
-    <origin xyz="0.00020722 0.0507 0.39997" rpy="0 0 0" />
-    <parent link="link2" />
-    <child link="link3" />
-    <axis xyz="0 1 0" />
-    <limit lower="-10" upper="10" effort="0" velocity="0" />
-  </joint>
-  <link name="link4">
-    <inertial>
-      <origin xyz="8.93211447726694E-05 -0.053367466841865 -0.0860702805514776" rpy="0 0 0" />
-      <mass value="0.284019990052222" />
-      <inertia ixx="0.0002676570674362" ixy="-3.02110627748532E-07" ixz="-4.10818936428236E-07" iyy="0.000253734082405407" iyz="-3.16043936161857E-05" izz="0.000344774781306503" />
-    </inertial>
-    <visual>
-      <origin xyz="0 0 0" rpy="0 0 0" />
-      <geometry>
-        <mesh filename="package://arm_description/meshes/link4.STL" />
-      </geometry>
-      <material name="">
-        <color rgba="0.792156862745098 0.819607843137255 0.933333333333333 1" />
-      </material>
-    </visual>
-    <collision>
-      <origin xyz="0 0 0" rpy="0 0 0" />
-      <geometry>
-        <mesh filename="package://arm_description/meshes/link4.STL" />
-      </geometry>
-    </collision>
-  </link>
-  <joint name="Joint4" type="revolute">
-    <origin xyz="-0.44676 0.035 0" rpy="0 0 0" />
-    <parent link="link3" />
-    <child link="link4" />
-    <axis xyz="0 -1 0" />
-    <limit lower="-10" upper="10" effort="0" velocity="0" />
-  </joint>
-  <link name="End_effector">
-    <inertial>
-      <origin xyz="-0.00291436016362501 -0.00153953625183378 -0.0697917938513681" rpy="0 0 0" />
-      <mass value="0.891224455695713" />
-      <inertia ixx="0.00266784691683874" ixy="-2.00928120275424E-06" ixz="1.12696986555021E-05" iyy="0.000652543524415568" iyz="-9.75739303299027E-06" izz="0.00233302824155854" />
-    </inertial>
-    <visual>
-      <origin xyz="0 0 0" rpy="0 0 0" />
-      <geometry>
-        <mesh filename="package://arm_description/meshes/End_effector.STL" />
-      </geometry>
-      <material name="">
-        <color rgba="0.792156862745098 0.819607843137255 0.933333333333333 1" />
-      </material>
-    </visual>
-    <collision>
-      <origin xyz="0 0 0" rpy="0 0 0" />
-      <geometry>
-        <mesh filename="package://arm_description/meshes/End_effector.STL" />
-      </geometry>
-    </collision>
-  </link>
-  <joint name="Joint5" type="revolute">
-    <origin xyz="0 -0.0617 -0.1125" rpy="0 0 0" />
-    <parent link="link4" />
-    <child link="End_effector" />
-    <axis xyz="0 0 -1" />
-    <limit lower="-10" upper="10" effort="0" velocity="0" />
-  </joint>
-  <xacro:arm_ros2_control
-    name="ExodusArmSystem"
-    use_fake_hardware="$(arg use_fake_hardware)"
-    can_interface="$(arg can_interface)"/>
 </robot>

Commit message: working Rviz gui operation including gripper operation needs a fix for servo node needs to add new URDF with full rover
Signed-off-by: TAUverIL <TAUverIL@gmail.com>

File: src/arm_controller/urdf/cubemars_test.ros2_control.urdf.xacro (robot description, xacro)
@@ -30,5 +30,5 @@
       <param name="vel_limit">5.03</param>
       <param name="trq_limit">120</param>
-      <param name="acc_limit">3.0</param>
+      <param name="acc_limit">10.0</param>
       <param name="enc_off">0.0</param>
       <param name="read_only">0</param>

File: src/arm_controller/urdf/dynamixel_test.ros2_control.urdf.xacro (robot description, xacro)
@@ -32,5 +32,5 @@
     <child link="Finger_Left"/>
     <axis xyz="-1 0 0"/>
-    <limit lower="0.0" upper="0.04" effort="7.3" velocity="5.55"/>
+    <limit lower="0.0" upper="0.08" effort="7.3" velocity="5.55"/>
   </joint>
   <joint name="Finger_Right_Joint" type="prismatic">
@@ -38,5 +38,5 @@
     <child link="Finger_Right"/>
     <axis xyz="1 0 0"/>
-    <limit lower="0.0" upper="0.04" effort="7.3" velocity="5.55"/>
+    <limit lower="0.0" upper="0.08" effort="7.3" velocity="5.55"/>
     <mimic joint="Finger_Left_Joint"/>
   </joint>

File: src/arm_description/urdf/AssemblyURDF_27.04.26.urdf (robot description, URDF)
Before this commit: robot AssemblyURDF_27.04.26, 8 links, 7 joints
Joints:
- joint Finger_Left_Joint: limit lower=0.0 upper=0.04 effort=7.3 velocity=5.55 -> lower=0.0 upper=0.08 effort=7.3 velocity=5.55
- joint Finger_Right_Joint: limit lower=0.0 upper=0.04 effort=7.3 velocity=5.55 -> lower=0.0 upper=0.08 effort=7.3 velocity=5.55

File: src/arm_description/urdf/arm.ros2_control.xacro (robot description, xacro)
@@ -33,8 +33,8 @@
         <param name="can_id">31</param>
         <param name="pole_pairs">21</param>
-        <param name="gear_ratio">1</param>
+        <param name="gear_ratio">64</param>
         <param name="kt">0.105</param>
         <param name="vel_limit">12.0</param>
-        <param name="acc_limit">3.0</param>
+        <param name="acc_limit">10.0</param>
         <param name="enc_off">0.0</param>
         <param name="direction">-1</param>
@@ -107,7 +107,7 @@
           <param name="id">1</param>
           <!-- Map MoveIt/URDF gripper travel to calibrated Dynamixel motor radians.
-               URDF: 0.0 = closed, 0.04 = open. Dynamixel: 0.5 = closed, -1.9 = open. -->
-          <param name="position_to_motor_scale">-60.0</param>
-          <param name="position_to_motor_offset">0.5</param>
+               URDF: 0.0 = closed, 0.08 = open. Dynamixel: -1.9 = closed, 2.9 = open. -->
+          <param name="position_to_motor_scale">60.0</param>
+          <param name="position_to_motor_offset">-1.9</param>
           <command_interface name="position"/>
           <state_interface name="position"/>
